File: kicadFiles/arcticPCB.sch (KiCad schematic (older format))
At the start: 262 parts, among them J1 USB_C_Receptacle, J2 Conn_01x04_Male, Q1 AO4406AL, SW1 MXSwitch, SW10 MXSwitch, SW11 MXSwitch, SW12 MXSwitch, SW13 MXSwitch, SW14 MXSwitch, SW15 MXSwitch, SW16 MXSwitch, SW17 MXSwitch, SW18 MXSwitch, SW19 MXSwitch, SW2 MXSwitch, SW20 MXSwitch, SW21 MXSwitch, SW22 MXSwitch, SW23 MXSwitch, SW24 MXSwitch, SW25 MXSwitch, SW26 MXSwitch, SW27 MXSwitch, SW28 MXSwitch, SW29 MXSwitch, SW3 MXSwitch, SW30 MXSwitch, SW31 MXSwitch, SW32 MXSwitch, SW33 MXSwitch, SW34 MXSwitch, SW35 MXSwitch, SW36 MXSwitch, SW37 MXSwitch, SW38 MXSwitch, SW39 MXSwitch, SW4 MXSwitch, SW40 MXSwitch, SW41 MXSwitch, SW42 MXSwitch, SW43 MXSwitch, SW44 MXSwitch, SW45 MXSwitch, SW46 MXSwitch, SW47 MXSwitch, SW48 MXSwitch, SW49 MXSwitch, SW5 MXSwitch, SW50 MXSwitch, SW51 MXSwitch, SW6 MXSwitch, SW7 MXSwitch, SW8 MXSwitch, SW9 MXSwitch, U1 STM32F303CCT6, U2 MCP1700-3302E_SOT23, Y1 8MHz

Commit message: [Update] Places some switches
Parts:
- removed C1, C2: 22p, Capacitor_SMD:C_0805_2012Metric_Pad1.15x1.40mm_HandSolder, symbol Device:C_Small
- removed C7, C9: 4.7n, Capacitor_SMD:C_0805_2012Metric_Pad1.15x1.40mm_HandSolder, symbol Device:C_Small
- removed CA1, CVBus2, CVBus3: 100n, Capacitor_SMD:C_0805_2012Metric_Pad1.15x1.40mm_HandSolder, symbol Device:C_Small
- removed CVBus4: 1u, Capacitor_SMD:C_0402_1005Metric, symbol Device:C_Small
- removed CVBus5: 4.7u, Capacitor_SMD:C_0805_2012Metric_Pad1.15x1.40mm_HandSolder, symbol Device:C_Small
- removed D42, D43, D44, D45, D46, D47, D48: 1N4148, acheronComponents:D_SOD-123, symbol Device:D
- removed DF1: RB060M-60TR, acheronComponents:D_SOD-123, symbol Device:D_Schottky_Small
- removed H7: CASE, MountingHole:MountingHole_2.2mm_M2_Pad_Via, symbol Mechanical:MountingHole_Pad
- removed J1: USB_C_Receptacle, USBconnector:TYPE-C-31-M-13, symbol Connector:USB_C_Receptacle
- removed J2: Conn_01x04_Male, acheronConnectors:JSTBM04B-ASRS, symbol Connector:Conn_01x04_Male
- removed L2: LogoBack, sharkLogo:skark, symbol Mechanical:MountingHole
- removed L4: BrazilianFlag, sharkLogo:brazilFlag, symbol Mechanical:MountingHole
- removed L5: usFlag, sharkLogo:usFlag, symbol Mechanical:MountingHole
- removed LED1, LED10, LED11, LED12, LED13, LED14, LED15, LED16, LED17, LED18, LED19, LED2, LED20, LED21, LED22, LED23, LED24, LED25, LED26, LED27, LED28, LED29, LED3, LED30, LED31, LED32, LED33, LED34, LED35, LED36, LED37, LED38, LED39, LED4, LED40, LED41, LED42, LED43, LED44, LED45, LED46, LED47, LED48, LED49, LED5, LED50, LED51, LED6, LED7, LED8, LED9: LED, acheronComponents:thtLED, symbol acheronSymbols:LED
- removed Q1: AO4406AL, acheronComponents:AO4406AL, symbol acheronSymbols:AO4406AL
- removed QRST1: BC847, Package_TO_SOT_SMD:SOT-23, symbol Transistor_BJT:BC847
- removed R5, R6: 1M, Resistor_SMD:R_1206_3216Metric_Pad1.42x1.75mm_HandSolder, symbol Device:R
- removed RA1, RA2, RB1, RB2, RPGate1: 10k, Resistor_SMD:R_1206_3216Metric_Pad1.42x1.75mm_HandSolder, symbol Device:R_Small
- removed RD+1, RD-1: 22R, Resistor_SMD:R_1206_3216Metric_Pad1.42x1.75mm_HandSolder, symbol Device:R_Small
- removed RD+Up1: 1.5k, Resistor_SMD:R_1206_3216Metric_Pad1.42x1.75mm_HandSolder, symbol Device:R_Small
- removed RGB1, RGB10, RGB2, RGB3, RGB4, RGB5, RGB6, RGB7, RGB8, RGB9: WS2812B, acheronComponents:LED_WS2812B, symbol LED:WS2812B
- removed RL1, RL10, RL11, RL12, RL13, RL14, RL15, RL16, RL17, RL18, RL19, RL2, RL20, RL21, RL22, RL23, RL24, RL25, RL26, RL27, RL28, RL29, RL3, RL30, RL31, RL32, RL33, RL34, RL35, RL36, RL37, RL38, RL39, RL40, RL41, RL42, RL43, RL44, RL45, RL46, RL47, RL48, RL5, RL6, RL7, RL8, RL9: 360, Resistor_SMD:R_1206_3216Metric, symbol Device:R_Small
- removed RL4: R_LED, Resistor_SMD:R_1206_3216Metric, symbol Device:R_Small
- removed ROT1, ROT2: Rotary_Encoder_Switch, acheronHardware:ALPS_EC11E, symbol Device:Rotary_Encoder_Switch
- removed RSGate1: 100, Resistor_SMD:R_1206_3216Metric_Pad1.42x1.75mm_HandSolder, symbol Device:R_Small
- removed SW42, SW43, SW44, SW45, SW46, SW47, SW48: MXSwitch, acheronKeyboardSwitches:MX100, symbol acheronSymbols:MXSwitch
- removed SW49, SW50, SW51: MXSwitch, acheronKeyboardSwitches:MX200R, symbol acheronSymbols:MXSwitch
- removed U1: STM32F303CCT6, Package_QFP:LQFP-48_7x7mm_P0.5mm, symbol acheronSymbols:STM32F303CCT6
- removed Y1: 8MHz, acheronComponents:Crystal_SMD_5032-4Pin_5.0x3.2mm, symbol Device:Crystal_GND24
- added CB2: 10n, Capacitor_SMD:C_0402_1005Metric, symbol Device:C_Small
- added CB3, CB8: 100n, Capacitor_SMD:C_0402_1005Metric, symbol Device:C_Small
- added CB4, CB6: 4.7uF, Capacitor_SMD:C_0402_1005Metric, symbol Device:C_Small
- added CB7: 100nF, Capacitor_SMD:C_0402_1005Metric, symbol Device:C_Small
- added CSH1: 4.7nF, Capacitor_SMD:C_0805_2012Metric, symbol Device:C_Small
- added CUSB1: 100n, Capacitor_SMD:C_0805_2012Metric_Pad1.15x1.40mm_HandSolder, symbol Device:C_Small
- added DF1: RB060M-60TR, acheron_Components:D_SOD-123, symbol Device:D_Schottky
- added H10, H7, H8, H9: Oval Mounting Hole, acheron_MountingHoles:MoutingHole_Oval_7mm_5.0x2.5mm, symbol Mechanical:MountingHole
- added J1: TYPE-C-31-M12_13, acheron_Connectors:TYPE-C-31-M-12, symbol acheronSymbols:TYPE-C-31-M12_13
- added J5: Conn_01x06_Male, acheron_Connectors:HEADER_6PIN_HORIZONTAL, symbol Connector:Conn_01x06_Male
- added L3: Label, SPV1_graphics:SPV1_preAlpha_Label_15x32mm, symbol Mechanical:MountingHole
- added QRST1: DTC123J, Package_TO_SOT_SMD:SOT-23, symbol Transistor_BJT:DTC123J
- added RSH1: 1M, acheron_Components:R_SMD_1026, symbol Device:R_Small
- added U1: STM32F072-LQFP48, acheron_Components:LQFP-48_7x7mm_P0.5mm, symbol acheronSymbols:STM32F072-LQFP48
- added U2: USBLC6-2SC6, acheron_Components:SOT-23-6, symbol Power_Protection:USBLC6-2SC6
- CB1: value 100n -> 1uF; footprint Capacitor_SMD:C_0805_2012Metric_Pad1.15x1.40mm_HandSolder -> Capacitor_SMD:C_0402_1005Metric
- CB5: renamed from CVBus1; footprint Capacitor_SMD:C_0805_2012Metric_Pad1.15x1.40mm_HandSolder -> Capacitor_SMD:C_0402_1005Metric
- CRST1: value 4.7n -> 10u
- D1, D10, D11, D12, D13, D14, D15, D16, D17, D18, D19, D2, D20, D21, D22, D23, D24, D25, D26, D27, D28, D29, D3, D30, D31, D32, D33, D34, D35, D36, D37, D38, D39, D4, D40, D41, D5, D6, D7, D8, D9: footprint acheronComponents:D_SOD-123 -> acheron_Components:D_SOD-123
- DRST1, DS1: footprint Diode_SMD:D_0805_2012Metric_Pad1.15x1.40mm_HandSolder -> acheron_Components:D_SOD-123
- F1: value 1A -> Polyfuse; footprint Fuse:Fuse_0805_2012Metric_Pad1.15x1.40mm_HandSolder -> acheron_Components:Fuse_1812_4532
- H1, H6: value MountingHole -> Half Side Hole; footprint MountingHole:MountingHole_2.5mm_Pad -> acheron_MountingHoles:halfSideHole
- H2: value MountingHole -> Mounting Hole; footprint MountingHole:MountingHole_2.5mm_Pad -> acheron_MountingHoles:MoutingHole_Oval_7mm_5.0x2.5mm
- H3, H4, H5: value MountingHole -> Oval Mounting Hole; footprint MountingHole:MountingHole_2.5mm_Pad -> acheron_MountingHoles:MoutingHole_Oval_7mm_5.0x2.5mm
- L1: value Logo -> Logos; footprint sharkLogo:sharkLogo -> SPV1_graphics:HxB_logo_10x36mm
- L2: renamed from L3; footprint sharkLogo:osh-logo -> oshLogo:osh-logo
- RCC1, RRST1: footprint Resistor_SMD:R_1206_3216Metric_Pad1.42x1.75mm_HandSolder -> acheron_Components:R_SMD_1026
- SW1, SW10, SW11, SW12, SW13, SW16, SW17, SW18, SW19, SW2, SW20, SW21, SW22, SW23, SW24, SW25, SW26, SW27, SW3, SW30, SW31, SW32, SW33, SW34, SW35, SW36, SW37, SW38, SW39, SW4, SW40, SW5, SW6, SW7, SW8, SW9: footprint acheronKeyboardSwitches:MX100 -> acheron_MX:MX100
- SW14: footprint acheronKeyboardSwitches:MX100 -> acheron_MX:MX200
- SW15, SW28: footprint acheronKeyboardSwitches:MX100 -> acheron_MX:MX150
- SW29: footprint acheronKeyboardSwitches:MX100 -> acheron_MX:MX175
- SW41: footprint acheronKeyboardSwitches:MX100 -> acheron_MX:MX225
- SWRST1: footprint smdPushBtn:smdPushBtn -> acheron_Hardware:smdPushBtn
- renumbered CSin1 to CSI1, CSout1 to CSO1, U2 to U3
Connections:
- net Row4 is gone; now on net Row3: D37.1 (K), D38.1 (K), D39.1 (K), D40.1 (K), D41.1 (K)
- net 3.3V: now also CB1.2, CB5.2, CB2.2, CB3.2, CB4.2, CB6.2, CB7.1, CB8.2, J5.6 (Pin_6), U1.1 (VBAT), U1.24 (VDD), U1.36 (VDDIO2), U1.48 (VDD), U1.9 (VDDA); no longer CB5.1
- net 5V: now also DF1.1 (K)
- net BOOT0: now also J5.3 (Pin_3), U1.44 (BOOT0)
- net Col1: now also SW15.1 (Col), SW29.1 (Col); no longer SW13.1 (Col), SW25.1 (Col), SW37.1 (Col)
- net Col10: now also SW24.1 (Col), SW38.1 (Col); no longer SW22.1 (Col), SW34.1 (Col)
- net Col11: now also SW25.1 (Col), SW39.1 (Col); no longer SW23.1 (Col), SW35.1 (Col)
- net Col12: now also SW26.1 (Col), SW40.1 (Col); no longer SW24.1 (Col), SW36.1 (Col)
- net Col2: now also SW16.1 (Col), SW30.1 (Col); no longer SW14.1 (Col), SW26.1 (Col), SW38.1 (Col)
- net Col3: now also SW17.1 (Col), SW31.1 (Col); no longer SW15.1 (Col), SW27.1 (Col), SW39.1 (Col)
- net Col4: now also SW18.1 (Col), SW32.1 (Col); no longer SW16.1 (Col), SW28.1 (Col), SW40.1 (Col)
- net Col5: now also SW19.1 (Col), SW33.1 (Col); no longer SW17.1 (Col), SW29.1 (Col), SW41.1 (Col)
- net Col6: now also SW20.1 (Col), SW34.1 (Col); no longer SW18.1 (Col), SW30.1 (Col)
- net Col7: now also SW21.1 (Col), SW35.1 (Col); no longer SW19.1 (Col), SW31.1 (Col)
- net Col8: now also SW22.1 (Col), SW36.1 (Col); no longer SW20.1 (Col), SW32.1 (Col)
- net Col9: now also SW23.1 (Col), SW37.1 (Col); no longer SW21.1 (Col), SW33.1 (Col)
- net D+: now also U1.33 (USB_DP/PA12), U2.3 (IO2)
- net D-: now also U1.32 (USB_DM/TIM1_CH4/PA11), U2.1 (IO1)
- net GND: now also CB5.1, CB2.1, CB3.1, CB4.1, CB6.1, CB7.2, CB8.1, CSH1.1, CUSB1.1, DF1.2 (A), J1.A1 (GND), J1.B1 (GND), J5.1 (Pin_1), QRST1.2 (E), RSH1.2, U1.23 (VSS), U1.35 (VSS), U1.47 (VSS), U1.8 (VSSA), U2.2 (GND); no longer CB5.2
- net NRST: now also J5.2 (Pin_2), QRST1.3 (C), U1.7 (NRST)
- net Row1: now also D13.1 (K), D14.1 (K)
- net Row2: now also D25.1 (K), D26.1 (K), D27.1 (K), D28.1 (K); no longer D13.1 (K), D14.1 (K), D15.1 (K)
- net Row3: no longer D25.1 (K), D26.1 (K), D27.1 (K), D28.1 (K), D29.1 (K)
- net VBUS: now also CUSB1.2, J1.A4 (VBUS), J1.B4 (VBUS), U2.5 (VBUS)
- net at RCC1.2: now also J1.A5 (CC1), J1.B5 (CC2)
- net at DRST1.2 (A), SWRST1.2: now also QRST1.1 (B)
- net EncS1: no longer names the net of D37.2 (A), SW37.2 (Row)
- new net Col13: SW13.1 (Col), SW27.1 (Col), SW41.1 (Col)
- new net Col14: SW14.1 (Col), SW28.1 (Col)
- new net DBus+: J1.A7 (D-), J1.B7 (D-), U2.4 (IO2)
- new net DBus-: J1.A6 (D+), J1.B6 (D+), U2.6 (IO1)
- new net SHIELD: CSH1.2, J1.S (SHIELD), RSH1.1
- new net SWCLK: J5.5 (Pin_5), U1.37 (SWCLK/PA14)
- new net SWDIO: J5.4 (Pin_4), U1.34 (SWDIO/PA13)
- no-connect marks 10 -> 2
Other:
- note added: "CBx are the bypass capacitors. Their value is specified in reference [2]."
- note added: "MCU"
- note added: "REFERENCES"
- note added: "Serial programming"
- note added: "Shield"
- note added: "USD ESD"
- note added: "[1] STM32F072x8 / STM32F072xB datasheet"
- note added: "[2] AN4080 Application note"
- note added: "https://www.st.com/content/ccc/resource/technical/document/application_note/c9/19/d7/b8/6b/0e/4c/d3/DM00051986.pdf/files/DM00051986.pdf/jcr:content/translations/en.DM00051986.pdf"
- note added: "https://www.st.com/resource/en/datasheet/stm32f072rb.pdf"
- note removed: "ESD\nProtection"
- note removed: "Encoder nets"
- note removed: "I2C Connector"
- note removed: "MCU and crystal"
- note removed: "Mounting holes"
- note removed: "Polyfuse PPTC RTC"
- note removed: "RGB"
- note removed: "Shield\nnet"
- note removed: "Switch LED matrix"
- note removed: "Switch matrix\n"
- note removed: "Voltage regulation\ncapacitor bank\n"
- moved on the sheet: CB5, CRST1, CRST2, CSI1, CSO1, D1, D10, D11, D12, D13, D2, D3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

Commit message: [Update] Finished placing switches, placed logo
Parts:
- added D42, D43, D44, D45, D46, D47, D48, D49, D50, D51, D52, D53, D54, D55, D56, D57, D58, D59, D60, D61, D65: 1N4148, acheron_Components:D_SOD-123, symbol Device:D
- added SW42: MXSwitch, acheron_MX:MX225, symbol acheronSymbols:MXSwitch
- added SW43, SW44, SW45, SW46, SW47, SW48, SW49, SW50, SW51, SW52, SW55, SW59, SW61, SW64, SW65: MXSwitch, acheron_MX:MX100, symbol acheronSymbols:MXSwitch
- added SW53: MXSwitch, acheron_MX:MX275, symbol acheronSymbols:MXSwitch
- added SW54, SW56, SW58, SW60: MXSwitch, acheron_MX:MX150, symbol acheronSymbols:MXSwitch
- added SW57: MXSwitch, acheron_MX:MX700R, symbol acheronSymbols:MXSwitch
- added SW62: MXSwitch, acheron_MX:MX175, symbol acheronSymbols:MXSwitch
- added SW63: MXSwitch, acheron_MX:MX125, symbol acheronSymbols:MXSwitch
Connections:
- net Col1: now also SW42.1 (Col), SW54.1 (Col), SW63.1 (Col)
- net Col10: now also SW51.1 (Col), SW59.1 (Col)
- net Col11: now also SW52.1 (Col), SW60.1 (Col)
- net Col12: now also SW53.1 (Col), SW62.1 (Col)
- net Col13: now also SW61.1 (Col)
- net Col14: now also SW64.1 (Col), SW65.1 (Col)
- net Col2: now also SW43.1 (Col), SW55.1 (Col)
- net Col3: now also SW44.1 (Col), SW56.1 (Col)
- net Col4: now also SW45.1 (Col)
- net Col5: now also SW46.1 (Col)
- net Col6: now also SW47.1 (Col)
- net Col7: now also SW48.1 (Col), SW57.1 (Col)
- net Col8: now also SW49.1 (Col)
- net Col9: now also SW50.1 (Col), SW58.1 (Col)
- net Row3: now also D29.1 (K), D65.1 (K)
- net at D14.2 (A), SW14.2 (Row): now also SW64.2 (Row)
- net at D29.2 (A), SW29.2 (Row): now also SW63.2 (Row)
- new net: D42.2 (A), SW42.2 (Row)
- new net: D43.2 (A), SW43.2 (Row)
- new net: D44.2 (A), SW44.2 (Row)
- new net: D45.2 (A), SW45.2 (Row)
- new net: D46.2 (A), SW46.2 (Row)
- new net: D47.2 (A), SW47.2 (Row)
- new net: D48.2 (A), SW48.2 (Row)
- new net: D49.2 (A), SW49.2 (Row)
- new net: D50.2 (A), SW50.2 (Row)
- new net: D51.2 (A), SW51.2 (Row)
- new net: D52.2 (A), SW52.2 (Row)
- new net: D53.2 (A), SW53.2 (Row), SW62.2 (Row)
- new net: D54.2 (A), SW54.2 (Row)
- new net: D55.2 (A), SW55.2 (Row)
- new net: D56.2 (A), SW56.2 (Row)
- new net: D57.2 (A), SW57.2 (Row)
- new net: D58.2 (A), SW58.2 (Row)
- new net: D59.2 (A), SW59.2 (Row)
- new net: D60.2 (A), SW60.2 (Row)
- new net: D61.2 (A), SW61.2 (Row)
- new net: D65.2 (A), SW65.2 (Row)
- new net Row4: D42.1 (K), D43.1 (K), D44.1 (K), D45.1 (K), D46.1 (K), D47.1 (K), D48.1 (K), D49.1 (K), D50.1 (K), D51.1 (K), D52.1 (K), D53.1 (K), D61.1 (K)
- new net Row5: D54.1 (K), D55.1 (K), D56.1 (K), D57.1 (K), D58.1 (K), D59.1 (K), D60.1 (K)
Other:
- note added: "SW14: 2U backspace"
- note added: "SW64: 1U left backspace"
- note added: "SW65: 1U right backspace"

Commit message: [Update,Feature] Added flex cuts, routed and placed most components
Parts:
- added J2, J3: Conn_01x06_Male, acheron_Connectors:HEADER_6PIN, symbol Connector:Conn_01x06_Male
- L1: value Logos -> ArcticLogo; footprint SPV1_graphics:HxB_logo_10x36mm -> arcticLogo:arcticLogoFilled
- L3: value Label -> Acheron Logo; footprint SPV1_graphics:SPV1_preAlpha_Label_15x32mm -> acheron_Logos:acheronLong
- renumbered D61 to D62
Connections:
- net 3.3V: now also J5.5 (Pin_5); no longer J5.6 (Pin_6)
- net Col10: now also SW58.1 (Col); no longer SW59.1 (Col)
- net Col11: now also SW59.1 (Col); no longer SW60.1 (Col)
- net Col12: now also SW60.1 (Col), SW61.1 (Col); no longer SW62.1 (Col)
- net Col13: now also SW62.1 (Col); no longer SW61.1 (Col)
- net Col9: no longer SW58.1 (Col)
- net GND: now also J5.6 (Pin_6); no longer J5.1 (Pin_1)
- net NRST: now also J5.1 (Pin_1); no longer J5.2 (Pin_2)
- net Row2: now also D15.1 (K)
- net SWCLK: now also J5.2 (Pin_2); no longer J5.5 (Pin_5)
- net J3_1: now reaches U1.20 (PB2)
- net J3_1: now also J3.1 (Pin_1)
- net J3_2: now reaches U1.21 (PB10/SPI2_SCK/I2C2_SCL/TIM2_CH3)
- net J3_2: now also J3.2 (Pin_2)
- net J3_3: now reaches U1.22 (PB11/TIM2_CH4/I2C2_SDA)
- net J3_3: now also J3.3 (Pin_3)
- net J3_4: now reaches U1.25 (PB12)
- net J3_4: now also J3.4 (Pin_4)
- net J3_5: now reaches U1.26 (SPI2_SCK/I2S2_CK/I2C2_SCL/PB13)
- net J3_5: now also J3.5 (Pin_5)
- net J3_6: now reaches U1.27 (PB14/SPI2_MISO/I2S2_MCK/I2C2_SDA/TIM15_CH1/PB15)
- net J3_6: now also J3.6 (Pin_6)
- net J2_1: now reaches U1.28 (SPI2_MOSI/I2S2_SD/PB15)
- net J2_1: now also J2.1 (Pin_1)
- net J2_2: now reaches U1.29 (TIM1_CH1/PA8)
- net J2_2: now also J2.2 (Pin_2)
- net J2_3: now reaches U1.30 (TIM1_CH2/PA9)
- net J2_3: now also J2.3 (Pin_3)
- net J2_4: now reaches U1.31 (TIM1_CH3/PA10)
- net J2_4: now also J2.4 (Pin_4)
- net J2_5: now reaches U1.38 (PA2)
- net J2_5: now also J2.5 (Pin_5)
- net J2_6: now reaches U1.39 (SPI1_SCK/I2S1_CK/TIM2_CH2/PB3)
- net J2_6: now also J2.6 (Pin_6)
- net at D53.2 (A), SW53.2 (Row): now also SW61.2 (Row); no longer SW62.2 (Row)
- net at D62.2 (A): now also SW62.2 (Row); no longer SW61.2 (Row)
Other:
- moved on the sheet: D58, D59, D60, SW58, SW59, SW60, SW61, SW62

Commit message: [Update] Finished routing
Connections:
- net 3.3V: now also J5.6 (Pin_6); no longer J5.5 (Pin_5)
- net BOOT0: now also J5.2 (Pin_2); no longer J5.3 (Pin_3)
- net GND: now also J5.5 (Pin_5); no longer J5.6 (Pin_6)
- net SWCLK: now also J5.3 (Pin_3); no longer J5.2 (Pin_2)
Changed lines of the file:
@@
 Text Notes 12725 14650 0    100  Italic 20
 Serial programming
-$Comp
-L power:GND #PWR0103
-U 1 1 5CFDFC6D
-P 13525 15725
-F 0 "#PWR0103" H 13525 15475 50  0001 C CNN
-F 1 "GND" V 13530 15597 50  0000 R CNN
-F 2 "" H 13525 15725 50  0001 C CNN
-F 3 "" H 13525 15725 50  0001 C CNN
-	1    13525 15725
-	0    -1   -1   0
-$EndComp
 Wire Wire Line
 	13525 15525 13450 15525
@@
 SWDIO
 Wire Wire Line
+	13450 15625 13525 15625
+Text GLabel 13525 15725 2    50   Input ~ 0
+3.3V
+Wire Wire Line
 	13450 15725 13525 15725
-Text GLabel 13525 15625 2    50   Input ~ 0
-3.3V
-Wire Wire Line
-	13450 15625 13525 15625
 Wire Wire Line
 	13525 15225 13450 15225
-Text GLabel 13525 15425 2    50   Input ~ 0
+Text GLabel 13525 15325 2    50   Input ~ 0
 BOOT0
 Text GLabel 13525 15225 2    50   Input ~ 0
 NRST
 Wire Wire Line
-	13450 15425 13525 15425
+	13450 15325 13525 15325
 $Comp
 L Transistor_BJT:DTC123J QRST1
@@
 	15925 7450 16925 7450
 Wire Wire Line
-	13450 15325 13525 15325
-Text GLabel 13525 15325 2    50   Input ~ 0
+	13450 15425 13525 15425
+Text GLabel 13525 15425 2    50   Input ~ 0
 SWCLK
 $Comp
@@
 	1    0    0    -1
 $EndComp
+$Comp
+L power:GND #PWR0103
+U 1 1 5CFDFC6D
+P 13525 15625
+F 0 "#PWR0103" H 13525 15375 50  0001 C CNN
+F 1 "GND" V 13530 15497 50  0000 R CNN
+F 2 "" H 13525 15625 50  0001 C CNN
+F 3 "" H 13525 15625 50  0001 C CNN
+	1    13525 15625
+	0    -1   -1   0
+$EndComp
 $EndSCHEMATC

Commit message: [Update] Finished routing
Connections:
- net Col1: now also U1.18 (PB0/TIM3_CH3/ADC_IN8)
- net Col10: now also U1.3 (PC14/OSC32_IN)
- net Col11: now also U1.2 (PC13)
- net Col12: now also U1.46 (SPI2_NSS/I2S2_WS/I2C1_SDA/TIM17_CH1/PB9)
- net Col13: now also U1.45 (I2C1_SCL/TIM16_CH1/PB8)
- net Col14: now also U1.43 (2C1_SDA/PB7)
- net Col2: now also U1.15 (PA5/ADC_IN5/DAC_OUT2)
- net Col3: now also U1.14 (PA4/TIM14_CH1/ADC_IN4)
- net Col4: now also U1.13 (PA3/TIM15_CH2/ADC_IN3)
- net Col5: now also U1.12 (PA2/ADC_IN2)
- net Col6: now also U1.11 (PA1/ADC_IN1)
- net Col7: now also U1.10 (PA0/ADC_IN0)
- net Col8: now also U1.6 (PF1/OSC_OUT)
- net Col9: now also U1.5 (PF0/OSC_IN)
- net Row1: now also U1.42 (I2C1_SCL/PB6)
- net Row2: now also U1.41 (SPI1_MOSI/I2S1_SD/TIM3_CH2/PB5)
- net Row3: now also U1.16 (PA6/ADC_IN6/TIM3_CH1/TIM16_CH1)
- net Row4: now also U1.17 (PA7/TIM3_CH2/TIM14_CH1/ADC_IN7)
- net Row5: now also U1.19 (PB1/TIM3_CH4/TIM14_CH1/ADC_IN9)
Changed lines of the file:
@@
 	0    -1   -1   0
 $EndComp
+Text GLabel 19250 19450 3    50   Input ~ 0
+Col3
+Wire Wire Line
+	19250 19450 19250 19400
+Text GLabel 19000 19450 3    50   Input ~ 0
+Col4
+Wire Wire Line
+	19000 19450 19000 19400
+Text GLabel 18600 19050 0    50   Input ~ 0
+Col5
+Wire Wire Line
+	18600 19050 18650 19050
+Text GLabel 18600 18800 0    50   Input ~ 0
+Col6
+Wire Wire Line
+	18600 18800 18650 18800
+Text GLabel 18600 18550 0    50   Input ~ 0
+Col7
+Wire Wire Line
+	18600 18550 18650 18550
+Text GLabel 18600 17550 0    50   Input ~ 0
+Col8
+Wire Wire Line
+	18600 17550 18650 17550
+Text GLabel 18600 17300 0    50   Input ~ 0
+Col9
+Wire Wire Line
+	18600 17300 18650 17300
+Text GLabel 18600 16800 0    50   Input ~ 0
+Col10
+Wire Wire Line
+	18600 16800 18650 16800
+Text GLabel 18600 16550 0    50   Input ~ 0
+Col11
+Wire Wire Line
+	18600 16550 18650 16550
+Text GLabel 19500 15900 1    50   Input ~ 0
+Col12
+Wire Wire Line
+	19500 15900 19500 15950
+Text GLabel 19750 15900 1    50   Input ~ 0
+Col13
+Wire Wire Line
+	19750 15900 19750 15950
+Text GLabel 20250 15900 1    50   Input ~ 0
+Col14
+Wire Wire Line
+	20250 15900 20250 15950
+Text GLabel 20500 15900 1    50   Input ~ 0
+Row1
+Wire Wire Line
+	20500 15900 20500 15950
+Text GLabel 19500 19450 3    50   Input ~ 0
+Col2
+Wire Wire Line
+	19500 19450 19500 19400
+Text GLabel 19750 19450 3    50   Input ~ 0
+Row3
+Wire Wire Line
+	19750 19450 19750 19400
+Text GLabel 20000 19450 3    50   Input ~ 0
+Row4
+Wire Wire Line
+	20000 19450 20000 19400
+Text GLabel 20500 19450 3    50   Input ~ 0
+Row5
+Wire Wire Line
+	20500 19450 20500 19400
+Text GLabel 20250 19450 3    50   Input ~ 0
+Col1
+Wire Wire Line
+	20250 19450 20250 19400
+Text GLabel 20750 15900 1    50   Input ~ 0
+Row2
+Wire Wire Line
+	20750 15900 20750 15950
 $EndSCHEMATC

Commit message: [Update] Added mounting holes ESD protection
Parts:
- added CSH2: 4.7nF, Capacitor_SMD:C_0805_2012Metric, symbol Device:C_Small
- added DSH1: 1N4007, acheron_Components:D_SOD-123, symbol Device:D
- added RSH2: 1M, acheron_Components:R_SMD_1026, symbol Device:R_Small
- H8: symbol Mechanical:MountingHole -> Mechanical:MountingHole_Pad
Connections:
- net GND: now also CSH2.1, RSH2.2
- new net: CSH2.2, DSH1.1 (K), RSH2.1
- new net CASE: DSH1.2 (A), H8.1
Other:
- note added: "Case ESD"
Changed lines of the file:
@@
 $EndComp
 $Comp
-L Mechanical:MountingHole H8
+L Mechanical:MountingHole_Pad H8
 U 1 1 5E63D4E1
-P 5250 19500
-F 0 "H8" H 5350 19546 50  0000 L CNN
-F 1 "Oval Mounting Hole" H 5350 19455 50  0000 L CNN
-F 2 "acheron_MountingHoles:MoutingHole_Oval_7mm_5.0x2.5mm" H 5250 19500 50  0001 C CNN
-F 3 "~" H 5250 19500 50  0001 C CNN
-	1    5250 19500
+P 6450 18050
+F 0 "H8" H 6550 18096 50  0000 L CNN
+F 1 "Oval Mounting Hole" H 6550 18005 50  0000 L CNN
+F 2 "acheron_MountingHoles:MoutingHole_Oval_7mm_5.0x2.5mm" H 6450 18050 50  0001 C CNN
+F 3 "~" H 6450 18050 50  0001 C CNN
+	1    6450 18050
 	1    0    0    -1
 $EndComp
@@
 Wire Wire Line
 	20750 15900 20750 15950
+$Comp
+L Device:R_Small RSH2
+U 1 1 5D45B6A0
+P 16200 15150
+F 0 "RSH2" H 16259 15181 31  0000 L CNN
+F 1 "1M" H 16259 15119 31  0000 L CNN
+F 2 "acheron_Components:R_SMD_1026" H 16200 15150 50  0001 C CNN
+F 3 "~" H 16200 15150 50  0001 C CNN
+	1    16200 15150
+	1    0    0    -1
+$EndComp
+$Comp
+L Device:C_Small CSH2
+U 1 1 5D45B6A6
+P 16075 15150
+F 0 "CSH2" V 16225 15150 31  0000 C CNN
+F 1 "4.7nF" V 16175 15150 31  0000 C CNN
+F 2 "Capacitor_SMD:C_0805_2012Metric" H 16075 15150 50  0001 C CNN
+F 3 "~" H 16075 15150 50  0001 C CNN
+	1    16075 15150
+	-1   0    0    1
+$EndComp
+Wire Wire Line
+	16200 15000 16200 15050
+Wire Wire Line
+	16075 15250 16075 15300
+Wire Wire Line
+	16075 15300 16200 15300
+Wire Wire Line
+	16200 15300 16200 15250
+Wire Wire Line
+	16200 15300 16200 15350
+Connection ~ 16200 15300
+$Comp
+L power:GND #PWR0111
+U 1 1 5D45B6B6
+P 16200 15350
+F 0 "#PWR0111" H 16200 15100 50  0001 C CNN
+F 1 "GND" H 16200 15225 31  0000 C CNN
+F 2 "" H 16200 15350 50  0001 C CNN
+F 3 "" H 16200 15350 50  0001 C CNN
+	1    16200 15350
+	1    0    0    -1
+$EndComp
+$Comp
+L Device:D DSH1
+U 1 1 5D48318C
+P 15725 15000
+F 0 "DSH1" V 15694 15079 31  0000 L CNN
+F 1 "1N4007" V 15756 15079 31  0000 L CNN
+F 2 "acheron_Components:D_SOD-123" H 15725 15000 50  0001 C CNN
+F 3 "~" H 15725 15000 50  0001 C CNN
+	1    15725 15000
+	-1   0    0    1
+$EndComp
+Text GLabel 15575 15000 0    50   Input ~ 0
+CASE
+Wire Notes Line width 20
+	15250 14500 16750 14500
+Wire Notes Line width 20
+	16750 14500 16750 16000
+Wire Notes Line width 20
+	16750 16000 15250 16000
+Wire Notes Line width 20
+	15250 14750 16750 14750
+Wire Notes Line width 20
+	15250 14500 15250 16000
+Text Notes 15600 14700 0    100  Italic 20
+Case ESD
+Wire Wire Line
+	15875 15000 16075 15000
+Wire Wire Line
+	16075 15050 16075 15000
+Connection ~ 16075 15000
+Wire Wire Line
+	16075 15000 16200 15000
+Text GLabel 6450 18150 3    50   Input ~ 0
+CASE
 $EndSCHEMATC
