File: kicadFiles/arcticPCB.kicad_pcb (KiCad board)
At the start: 2 copper layers, 285 x 94 mm, 7 parts, among them J1 TYPE-C-31-M-12

Commit message: [Update] Places some switches
Parts:
- removed HOLE: H1, acheronMountingHoles:ovalHole
- removed HOLE: H6, acheronMountingHoles:ovalHole
- removed HOLE: H4, acheronMountingHoles:ovalHole
- removed HOLE: H2, acheronMountingHoles:singleHole
- added CB1: 1uF, Capacitor_SMD:C_0402_1005Metric, F.Cu at (191.0, -189.0)
- added CB2: 10n, Capacitor_SMD:C_0402_1005Metric, F.Cu at (202.3, -201.1)
- added CB3: 100n, Capacitor_SMD:C_0402_1005Metric, F.Cu at (202.3, -203.1)
- added CB4: 4.7uF, Capacitor_SMD:C_0402_1005Metric, F.Cu at (202.3, -205.1)
- added CB5: 100n, Capacitor_SMD:C_0402_1005Metric, F.Cu at (202.3, -207.1)
- added CB6: 4.7uF, Capacitor_SMD:C_0402_1005Metric, F.Cu at (202.3, -199.1)
- added CB7: 100nF, Capacitor_SMD:C_0402_1005Metric, F.Cu at (313.4, -308.0)
- added CB8: 100n, Capacitor_SMD:C_0402_1005Metric, F.Cu at (316.3, -308.0)
- added CRST1: 10u, Capacitor_SMD:C_0805_2012Metric_Pad1.15x1.40mm_HandSolder, F.Cu at (215.7, -258.6)
- added CRST2: 4.7n, Capacitor_SMD:C_0805_2012Metric_Pad1.15x1.40mm_HandSolder, F.Cu at (215.7, -261.5)
- added CSH1: 4.7nF, Capacitor_SMD:C_0805_2012Metric, F.Cu at (199.0, -230.1)
- added CSI1: 100n, Capacitor_SMD:C_0805_2012Metric_Pad1.15x1.40mm_HandSolder, F.Cu at (215.7, -267.4)
- added CSO1: 100n, Capacitor_SMD:C_0805_2012Metric_Pad1.15x1.40mm_HandSolder, F.Cu at (215.7, -264.5)
- added CUSB1: 100n, Capacitor_SMD:C_0805_2012Metric_Pad1.15x1.40mm_HandSolder, F.Cu at (215.7, -270.4)
- added D1: 1N4148, acheron_Components:D_SOD-123, F.Cu at (476.1, -285.7)
- added D10: 1N4148, acheron_Components:D_SOD-123, F.Cu at (414.2, -225.3)
- added D11: 1N4148, acheron_Components:D_SOD-123, F.Cu at (432.1, -242.1)
- added D12: 1N4148, acheron_Components:D_SOD-123, F.Cu at (443.8, -255.5)
- added D13: 1N4148, acheron_Components:D_SOD-123, F.Cu at (414.2, -232.0)
- added D14: 1N4148, acheron_Components:D_SOD-123, F.Cu at (130.6, -177.7)
- added D15: 1N4148, acheron_Components:D_SOD-123, F.Cu at (415.2, -34.9)
- added D16: 1N4148, acheron_Components:D_SOD-123, F.Cu at (348.9, -14.7)
- added D17: 1N4148, acheron_Components:D_SOD-123, F.Cu at (354.7, -14.7)
- added D18: 1N4148, acheron_Components:D_SOD-123, F.Cu at (360.6, -14.7)
- added D19: 1N4148, acheron_Components:D_SOD-123, F.Cu at (366.4, -14.7)
- added D2: 1N4148, acheron_Components:D_SOD-123, F.Cu at (443.8, -252.1)
- added D20: 1N4148, acheron_Components:D_SOD-123, F.Cu at (372.3, -14.7)
- added D21: 1N4148, acheron_Components:D_SOD-123, F.Cu at (378.1, -14.7)
- added D22: 1N4148, acheron_Components:D_SOD-123, F.Cu at (384.0, -14.7)
- added D23: 1N4148, acheron_Components:D_SOD-123, F.Cu at (409.3, -34.9)
- added D24: 1N4148, acheron_Components:D_SOD-123, F.Cu at (429.5, -55.0)
- added D25: 1N4148, acheron_Components:D_SOD-123, F.Cu at (435.3, -55.0)
- added D26: 1N4148, acheron_Components:D_SOD-123, F.Cu at (429.5, -51.7)
- added D27: 1N4148, acheron_Components:D_SOD-123, F.Cu at (-52.8, -40.8)
- added D28: 1N4148, acheron_Components:D_SOD-123, F.Cu at (-46.9, -40.8)
- added D29: 1N4148, acheron_Components:D_SOD-123, F.Cu at (466.9, 16.0)
- added D3: 1N4148, acheron_Components:D_SOD-123, F.Cu at (476.1, -289.1)
- added D30: 1N4148, acheron_Components:D_SOD-123, F.Cu at (362.5, 71.7)
- added D31: 1N4148, acheron_Components:D_SOD-123, F.Cu at (368.4, 71.7)
- added D32: 1N4148, acheron_Components:D_SOD-123, F.Cu at (374.2, 71.7)
- added D33: 1N4148, acheron_Components:D_SOD-123, F.Cu at (380.1, 71.7)
- added D34: 1N4148, acheron_Components:D_SOD-123, F.Cu at (385.9, 71.7)
- added D35: 1N4148, acheron_Components:D_SOD-123, F.Cu at (391.8, 71.7)
- added D36: 1N4148, acheron_Components:D_SOD-123, F.Cu at (397.6, 71.7)
- added D37: 1N4148, acheron_Components:D_SOD-123, F.Cu at (403.5, 71.7)
- added D38: 1N4148, acheron_Components:D_SOD-123, F.Cu at (466.9, 9.30)
- added D39: 1N4148, acheron_Components:D_SOD-123, F.Cu at (472.8, 9.30)
- added D4: 1N4148, acheron_Components:D_SOD-123, F.Cu at (481.9, -292.4)
- added D40: 1N4148, acheron_Components:D_SOD-123, F.Cu at (466.9, 12.7)
- added D41: 1N4148, acheron_Components:D_SOD-123, F.Cu at (472.8, 12.7)
- added D42: 1N4148, acheron_Components:D_SOD-123, F.Cu at (-84.5, 133.2)
- added D43: 1N4148, acheron_Components:D_SOD-123, F.Cu at (-114.1, 135.1)
- added D44: 1N4148, acheron_Components:D_SOD-123, F.Cu at (-108.3, 135.1)
- added D45: 1N4148, acheron_Components:D_SOD-123, F.Cu at (-70.2, 113.0)
- added D46: 1N4148, acheron_Components:D_SOD-123, F.Cu at (-102.4, 135.1)
- added D47: 1N4148, acheron_Components:D_SOD-123, F.Cu at (-50.0, 92.9)
- added D48: 1N4148, acheron_Components:D_SOD-123, F.Cu at (-96.6, 135.1)
- added D49: 1N4148, acheron_Components:D_SOD-123, F.Cu at (-90.3, 133.2)
- added D5: 1N4148, acheron_Components:D_SOD-123, F.Cu at (335.8, -146.4)
- added D50: 1N4148, acheron_Components:D_SOD-123, F.Cu at (-70.2, 116.4)
- added D51: 1N4148, acheron_Components:D_SOD-123, F.Cu at (-64.3, 113.0)
- added D52: 1N4148, acheron_Components:D_SOD-123, F.Cu at (-50.0, 96.2)
- added D53: 1N4148, acheron_Components:D_SOD-123, F.Cu at (-44.1, 92.9)
- added D54: 1N4148, acheron_Components:D_SOD-123, F.Cu at (85.3, 185.4)
- added D55: 1N4148, acheron_Components:D_SOD-123, F.Cu at (105.5, 165.3)
- added D56: 1N4148, acheron_Components:D_SOD-123, F.Cu at (85.3, 188.8)
- added D57: 1N4148, acheron_Components:D_SOD-123, F.Cu at (77.0, 105.6)
- added D58: 1N4148, acheron_Components:D_SOD-123, F.Cu at (247.3, 150.9)
- added D59: 1N4148, acheron_Components:D_SOD-123, F.Cu at (267.4, 130.7)
- added D6: 1N4148, acheron_Components:D_SOD-123, F.Cu at (425.9, -235.3)
- added D60: 1N4148, acheron_Components:D_SOD-123, F.Cu at (247.3, 154.2)
- added D7: 1N4148, acheron_Components:D_SOD-123, F.Cu at (408.3, -218.6)
- added D8: 1N4148, acheron_Components:D_SOD-123, F.Cu at (420.0, -232.0)
- added D9: 1N4148, acheron_Components:D_SOD-123, F.Cu at (408.3, -221.9)
- added DF1: RB060M-60TR, acheron_Components:D_SOD-123, F.Cu at (290.9, -146.1)
- added DRST1: 1N4148, acheron_Components:D_SOD-123, F.Cu at (432.1, -255.5)
- added DS1: 1N4148, acheron_Components:D_SOD-123, F.Cu at (408.3, -232.0)
- added F1: Polyfuse, acheron_Components:Fuse_1812_4532, F.Cu at (335.5, -298.3)
- added H1: Half Side Hole, acheron_MountingHoles:halfSideHole, B.Cu at (285.0, 56.5)
- added H10: Oval Mounting Hole, acheron_MountingHoles:MoutingHole_Oval_7mm_5.0x2.5mm, F.Cu at (75.8, 9.20)
- added H3: Oval Mounting Hole, acheron_MountingHoles:MoutingHole_Oval_7mm_5.0x2.5mm, B.Cu at (156.8, 47.3)
- added H4: Oval Mounting Hole, acheron_MountingHoles:MoutingHole_Oval_7mm_5.0x2.5mm, B.Cu at (94.5, 85.2)
- added H6: Half Side Hole, acheron_MountingHoles:halfSideHole, B.Cu at (0.00, 56.5)
- added H7: Oval Mounting Hole, acheron_MountingHoles:MoutingHole_Oval_7mm_5.0x2.5mm, F.Cu at (260.9, 85.2)
- added H8: Oval Mounting Hole, acheron_MountingHoles:MoutingHole_Oval_7mm_5.0x2.5mm, F.Cu at (209.2, 9.20)
- added H9: Oval Mounting Hole, acheron_MountingHoles:MoutingHole_Oval_7mm_5.0x2.5mm, F.Cu at (25.6, 89.0)
- added J5: Conn_01x06_Male, acheron_Connectors:HEADER_6PIN_HORIZONTAL, F.Cu at (336.4, -303.9)
- added L2: OSHLogo, oshLogo:osh-logo, F.Cu at (186.6, 56.8)
- added QRST1: DTC123J, Package_TO_SOT_SMD:SOT-23, F.Cu at (215.6, -254.8)
- added RCC1: 5.1k, acheron_Components:R_SMD_1026, F.Cu at (193.8, -229.9)
- added RRST1: 100k, acheron_Components:R_SMD_1026, F.Cu at (187.8, -229.9)
- added RSH1: 1M, acheron_Components:R_SMD_1026, F.Cu at (181.9, -229.9)
- added SW1: MXSwitch, acheron_MX:MX100, F.Cu at (275.9, 9.20)
- added SW10: MXSwitch, acheron_MX:MX100, F.Cu at (104.4, 9.20)
- added SW11: MXSwitch, acheron_MX:MX100, F.Cu at (85.3, 9.20)
- added SW12: MXSwitch, acheron_MX:MX100, F.Cu at (66.3, 9.20)
- added SW13: MXSwitch, acheron_MX:MX100, F.Cu at (47.2, 9.20)
- added SW14: MXSwitch, acheron_MX:MX200, F.Cu at (18.7, 9.20)
- added SW15: MXSwitch, acheron_MX:MX150, F.Cu at (271.1, 28.3)
- added SW16: MXSwitch, acheron_MX:MX100, F.Cu at (247.3, 28.3)
- added SW17: MXSwitch, acheron_MX:MX100, F.Cu at (228.2, 28.3)
- added SW18: MXSwitch, acheron_MX:MX100, F.Cu at (209.2, 28.3)
- added SW19: MXSwitch, acheron_MX:MX100, F.Cu at (190.1, 28.3)
- added SW2: MXSwitch, acheron_MX:MX100, F.Cu at (256.8, 9.20)
- added SW20: MXSwitch, acheron_MX:MX100, F.Cu at (171.1, 28.3)
- added SW21: MXSwitch, acheron_MX:MX100, F.Cu at (152.0, 28.3)
- added SW22: MXSwitch, acheron_MX:MX100, F.Cu at (133.0, 28.3)
- added SW23: MXSwitch, acheron_MX:MX100, F.Cu at (113.9, 28.3)
- added SW24: MXSwitch, acheron_MX:MX100, F.Cu at (94.9, 28.3)
- added SW25: MXSwitch, acheron_MX:MX100, F.Cu at (75.8, 28.3)
- added SW26: MXSwitch, acheron_MX:MX100, F.Cu at (56.8, 28.3)
- added SW27: MXSwitch, acheron_MX:MX100, F.Cu at (37.7, 28.3)
- added SW28: MXSwitch, acheron_MX:MX150, F.Cu at (13.9, 28.3)
- added SW29: MXSwitch, acheron_MX:MX175, F.Cu at (268.7, 47.3)
- added SW3: MXSwitch, acheron_MX:MX100, F.Cu at (237.7, 9.20)
- added SW30: MXSwitch, acheron_MX:MX100, F.Cu at (242.5, 47.3)
- added SW31: MXSwitch, acheron_MX:MX100, F.Cu at (223.5, 47.3)
- added SW32: MXSwitch, acheron_MX:MX100, F.Cu at (204.4, 47.3)
- added SW33: MXSwitch, acheron_MX:MX100, F.Cu at (185.4, 47.3)
- added SW34: MXSwitch, acheron_MX:MX100, F.Cu at (166.3, 47.3)
- added SW35: MXSwitch, acheron_MX:MX100, F.Cu at (147.3, 47.3)
- added SW36: MXSwitch, acheron_MX:MX100, F.Cu at (128.2, 47.3)
- added SW37: MXSwitch, acheron_MX:MX100, F.Cu at (109.2, 47.3)
- added SW38: MXSwitch, acheron_MX:MX100, F.Cu at (90.1, 47.3)
- added SW39: MXSwitch, acheron_MX:MX100, F.Cu at (71.1, 47.3)
- added SW4: MXSwitch, acheron_MX:MX100, F.Cu at (218.7, 9.20)
- added SW40: MXSwitch, acheron_MX:MX100, F.Cu at (52.0, 47.3)
- added SW41: MXSwitch, acheron_MX:MX225, F.Cu at (21.1, 47.3)
- added SW42: MXSwitch, acheron_MX:MX225, F.Cu at (263.9, 66.4)
- added SW43: MXSwitch, acheron_MX:MX100, F.Cu at (233.0, 66.4)
- added SW44: MXSwitch, acheron_MX:MX100, F.Cu at (213.9, 66.4)
- added SW45: MXSwitch, acheron_MX:MX100, F.Cu at (194.9, 66.4)
- added SW46: MXSwitch, acheron_MX:MX100, F.Cu at (175.8, 66.4)
- added SW47: MXSwitch, acheron_MX:MX100, F.Cu at (156.8, 66.4)
- added SW48: MXSwitch, acheron_MX:MX100, F.Cu at (137.7, 66.4)
- added SW49: MXSwitch, acheron_MX:MX100, F.Cu at (118.7, 66.4)
- added SW5: MXSwitch, acheron_MX:MX100, F.Cu at (199.6, 9.20)
- added SW50: MXSwitch, acheron_MX:MX100, F.Cu at (99.6, 66.4)
- added SW51: MXSwitch, acheron_MX:MX100, F.Cu at (80.6, 66.4)
- added SW52: MXSwitch, acheron_MX:MX100, F.Cu at (61.5, 66.4)
- added SW53: MXSwitch, acheron_MX:MX275, F.Cu at (25.8, 66.4)
- added SW54: MXSwitch, acheron_MX:MX150, F.Cu at (13.9, 85.4)
- added SW55: MXSwitch, acheron_MX:MX100, F.Cu at (37.7, 85.4)
- added SW56: MXSwitch, acheron_MX:MX150, F.Cu at (61.5, 85.4)
- added SW57: MXSwitch, acheron_MX:MX700R, F.Cu at (142.5, 85.4)
- added SW58: MXSwitch, acheron_MX:MX150, F.Cu at (223.5, 85.4)
- added SW59: MXSwitch, acheron_MX:MX100, F.Cu at (247.3, 85.4)
- added SW6: MXSwitch, acheron_MX:MX100, F.Cu at (180.6, 9.20)
- added SW60: MXSwitch, acheron_MX:MX150, F.Cu at (271.1, 85.4)
- added SW7: MXSwitch, acheron_MX:MX100, F.Cu at (161.5, 9.20)
- added SW8: MXSwitch, acheron_MX:MX100, F.Cu at (142.5, 9.20)
- added SW9: MXSwitch, acheron_MX:MX100, F.Cu at (123.4, 9.20)
- added SWRST1: SW_Push, acheron_Hardware:smdPushBtn, F.Cu at (194.3, -193.4)
- added U1: STM32F072-LQFP48, acheron_Components:LQFP-48_7x7mm_P0.5mm, F.Cu at (255.6, 37.8)
- added U2: USBLC6-2SC6, acheron_Components:SOT-23-6, F.Cu at (463.4, -270.9)
- added U3: MCP1700-3302E_SOT23, Package_TO_SOT_SMD:SOT-23, F.Cu at (201.3, -194.5)
- H2: value LOGO -> Mounting Hole; footprint acheronMountingHoles:halfSideHole -> acheron_MountingHoles:MoutingHole_Oval_7mm_5.0x2.5mm; moved to B.Cu
- H5: value LOGO -> Oval Mounting Hole; footprint acheronMountingHoles:halfSideHole -> acheron_MountingHoles:MoutingHole_Oval_7mm_5.0x2.5mm; moved to B.Cu
- J1: value TYPE-C-31-M-12 -> TYPE-C-31-M12_13; footprint acheronConnectors:TYPE-C-31-M-12 -> acheron_Connectors:TYPE-C-31-M-12; moved to F.Cu
- moved H5 261.6 mm to (25.0, 28.0)
- moved H2 261.4 mm to (259.8, 27.9), turned to 180 degrees
- moved J1 252.6 mm to (266.8, 5.70), turned to 180 degrees
Connections:
- J1 pad A1: (no net) -> GND
- J1 pad A4: (no net) -> VBUS
- J1 pad A5: (no net) -> Net-(J1-PadA5)
- J1 pad A6: (no net) -> DBus-
- J1 pad A7: (no net) -> DBus+
- J1 pad A8: (no net) -> Net-(J1-PadA8)
- J1 pad B1: (no net) -> GND
- J1 pad B4: (no net) -> VBUS
- J1 pad B5: (no net) -> Net-(J1-PadA5)
- J1 pad B6: (no net) -> DBus-
- J1 pad B7: (no net) -> DBus+
- J1 pad B8: (no net) -> Net-(J1-PadB8)
Routing:
- net (no net): vias 0 -> 1

Commit message: [Update] Finished placing switches, placed logo
Parts:
- added D61: 1N4148, acheron_Components:D_SOD-123, F.Cu at (-102.8, 62.8)
- added D65: 1N4148, acheron_Components:D_SOD-123, F.Cu at (-68.2, 3.25)
- added G***: LOGO, arcticLogo:arcticLogoFilled, B.Cu at (118.7, 84.2)
- added SW61: MXSwitch, acheron_MX:MX100, F.Cu at (42.5, 66.4)
- added SW62: MXSwitch, acheron_MX:MX175, F.Cu at (16.3, 66.4)
- added SW63: MXSwitch, acheron_MX:MX125, F.Cu at (273.5, 47.3)
- added SW64: MXSwitch, acheron_MX:MX100, F.Cu at (28.2, 9.20)
- added SW65: MXSwitch, acheron_MX:MX100, F.Cu at (9.15, 9.20)
- moved J1 2.18 mm to (267.4, 7.80)
- moved H1 1.06 mm to (284.0, 56.8)
- moved H6 1.05 mm to (1.00, 56.8)
- moved H2 0.67 mm to (260.4, 28.3)
- moved H5 0.25 mm to (25.0, 28.3)
- moved H9 0.23 mm to (25.6, 88.8)
Other:
- board size 285 x 94 mm -> 283 x 94.2 mm

Commit message: [Update] Added 1mm clearance to mounting holes and added ground planes
Parts:
- moved L2 5.54 mm to (191.8, 55.2)
Routing:
- net GND: track 0.00 -> 1.67 mm, vias 0 -> 1
- added copper zone on B.Cu, net GND
- added copper zone on F.Cu, net GND
Changed lines of the file:
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@@
     (thickness 1.6)
     (drawings 30)
-    (tracks 1)
+    (tracks 3)
     (zones 0)
     (modules 167)
@@
     (last_trace_width 0.25)
     (trace_clearance 0.2)
-    (zone_clearance 0.508)
+    (zone_clearance 0.254)
     (zone_45_only no)
     (trace_min 0.2)
@@
     (mod_text_size 1 1)
     (mod_text_width 0.15)
-    (pad_size 2.54 2.54)
-    (pad_drill 1.525)
+    (pad_size 6.5 4)
+    (pad_drill 5)
     (pad_to_mask_clearance 0.051)
     (solder_mask_min_width 0.25)
@@
       (effects (font (size 1 1) (thickness 0.15)) (justify mirror))
     )
-    (pad 1 thru_hole oval (at 0 0 180) (size 6.5 4) (drill oval 5 2.5) (layers *.Cu *.Mask))
+    (pad 1 thru_hole oval (at 0 0 180) (size 6.5 4) (drill oval 5 2.5) (layers *.Cu *.Mask)
+      (clearance 1))
     (model cherry_mx1.wrl
       (at (xyz 0 0 0))
@@
       (effects (font (size 1.524 1.524) (thickness 0.3048)))
     )
-    (pad 1 thru_hole oval (at 0 0) (size 6.5 4) (drill oval 5 2.5) (layers *.Cu *.Mask))
+    (pad 1 thru_hole oval (at 0 0) (size 6.5 4) (drill oval 5 2.5) (layers *.Cu *.Mask)
+      (clearance 1))
     (model cherry_mx1.wrl
       (at (xyz 0 0 0))
@@
       (effects (font (size 1.524 1.524) (thickness 0.3048)))
     )
-    (pad 1 thru_hole oval (at -3.55 0.2) (size 6.5 4) (drill oval 5 2.5) (layers *.Cu *.Mask))
+    (pad 1 thru_hole oval (at -3.55 0.2) (size 6.5 4) (drill oval 5 2.5) (layers *.Cu *.Mask)
+      (clearance 1))
     (model cherry_mx1.wrl
       (at (xyz 0 0 0))
@@
       (effects (font (size 1.524 1.524) (thickness 0.3048)))
     )
-    (pad 1 thru_hole oval (at 0 0) (size 6.5 4) (drill oval 5 2.5) (layers *.Cu *.Mask))
+    (pad 1 thru_hole oval (at 0 0) (size 6.5 4) (drill oval 5 2.5) (layers *.Cu *.Mask)
+      (clearance 1))
     (model cherry_mx1.wrl
       (at (xyz 0 0 0))
@@
       (effects (font (size 1.524 1.524) (thickness 0.3048)))
     )
-    (pad 1 thru_hole oval (at 0 0) (size 6.5 4) (drill oval 5 2.5) (layers *.Cu *.Mask))
+    (pad 1 thru_hole oval (at 0 0) (size 6.5 4) (drill oval 5 2.5) (layers *.Cu *.Mask)
+      (clearance 1))
     (model cherry_mx1.wrl
       (at (xyz 0 0 0))
@@
       (effects (font (size 1.524 1.524) (thickness 0.3048)) (justify mirror))
     )
-    (pad 1 thru_hole oval (at 0 0 180) (size 6.5 4) (drill oval 5 2.5) (layers *.Cu *.Mask))
+    (pad 1 thru_hole oval (at 0 0 180) (size 6.5 4) (drill oval 5 2.5) (layers *.Cu *.Mask)
+      (clearance 1))
     (model cherry_mx1.wrl
       (at (xyz 0 0 0))
@@
       (effects (font (size 1.524 1.524) (thickness 0.3048)) (justify mirror))
     )
-    (pad 1 thru_hole oval (at 0 0 180) (size 6.5 4) (drill oval 5 2.5) (layers *.Cu *.Mask))
+    (pad 1 thru_hole oval (at 0 0 180) (size 6.5 4) (drill oval 5 2.5) (layers *.Cu *.Mask)
+      (clearance 1))
     (model cherry_mx1.wrl
       (at (xyz 0 0 0))
@@
       (effects (font (size 1.524 1.524) (thickness 0.3048)) (justify mirror))
     )
-    (pad 1 thru_hole oval (at 0 0 180) (size 6.5 4) (drill oval 5 2.5) (layers *.Cu *.Mask))
+    (pad 1 thru_hole oval (at 0 0 180) (size 6.5 4) (drill oval 5 2.5) (layers *.Cu *.Mask)
+      (clearance 1))
     (model cherry_mx1.wrl
       (at (xyz 0 0 0))
@@
     (fp_line (start -6 0) (end 6 0) (layer Cmts.User) (width 0.1))
     (fp_line (start 0 4) (end 0 -4) (layer Cmts.User) (width 0.1))
-    (pad "" thru_hole oval (at 0 0 180) (size 10 4.5) (drill oval 8 2.5) (layers *.Cu *.Mask))
+    (pad "" thru_hole oval (at 0 0 180) (size 10 4.5) (drill oval 8 2.5) (layers *.Cu *.Mask)
+      (clearance 1))
   )
   (module acheron_MountingHoles:halfSideHole (layer B.Cu)
@@
     (fp_line (start -6 0) (end 6 0) (layer Cmts.User) (width 0.1))
     (fp_line (start 0 4) (end 0 -4) (layer Cmts.User) (width 0.1))
-    (pad "" thru_hole oval (at 0 0) (size 10 4.5) (drill oval 8 2.5) (layers *.Cu *.Mask))
+    (pad "" thru_hole oval (at 0 0) (size 10 4.5) (drill oval 8 2.5) (layers *.Cu *.Mask)
+      (clearance 1))
   )
   (module acheron_MX:MX225 (layer F.Cu)
@@
   )
   (module oshLogo:osh-logo (layer F.Cu)
-    (at 186.55275 56.8252)
+    (at 191.85 55.2)
     (fp_text reference L2 (at 0 0) (layer F.SilkS) hide
       (effects (font (size 1.524 1.524) (thickness 0.3)))
@@
   (gr_line (start 4 0.2) (end 281 0.2) (layer Edge.Cuts) (width 0.2))
   (via (at 22.825 110.05) (size 0.8) (drill 0.4) (layers F.Cu B.Cu) (net 0))
+  (segment (start 264.15 6.525) (end 264.15 8.2) (width 0.25) (layer F.Cu) (net 2))
+  (via (at 264.15 9.2) (size 1) (drill 0.5) (layers F.Cu B.Cu) (net 2))
   (zone (net 0) (net_name "") (layer F.Cu) (hatch edge 0.508)
     (connect_pads (clearance 0.508))
@@
     (polygon
       (pts
-        (xy 262.65 1) (xy 262.65 6.4) (xy 271.75 6.4) (xy 271.75 1)
+        (xy 262.65 1) (xy 262.65 5.95) (xy 271.75 5.95) (xy 271.75 1)
+      )
+    )
+  )
+  (zone (net 2) (net_name GND) (layer F.Cu) (hatch edge 0.508)
+    (connect_pads yes (clearance 0.254))
+    (min_thickness 0.127)
+    (fill yes (arc_segments 32) (thermal_gap 0.508) (thermal_bridge_width 0.508))
+    (polygon
+      (pts
+        (xy -0.15 -0.8) (xy 284.85 -0.8) (xy 284.85 95.2) (xy -0.15 95.2)
+      )
+    )
+  )
+  (zone (net 2) (net_name GND) (layer B.Cu) (hatch edge 0.508)
+    (connect_pads yes (clearance 0.254))
+    (min_thickness 0.127)
+    (fill yes (arc_segments 32) (thermal_gap 0.508) (thermal_bridge_width 0.508) (smoothing fillet))
+    (polygon
+      (pts
+        (xy -1.15 -1.8) (xy 285.85 -1.8) (xy 285.85 96.2) (xy -1.15 96.2)
       )
     )

Commit message: [Update,Feature] Added flex cuts, routed and placed most components
Parts:
- removed G***: LOGO, arcticLogo:arcticLogoFilled
- added J2: Conn_01x06_Male, acheron_Connectors:HEADER_6PIN, F.Cu at (282.2, 25.7)
- added J3: Conn_01x06_Male, acheron_Connectors:HEADER_6PIN, F.Cu at (282.2, 41.0)
- added L1: ArcticLogo, arcticLogo:arcticLogoFilled, B.Cu at (121.1, 85.4)
- added L3: Acheron Logo, acheron_Logos:acheronLong, F.Cu at (177.0, 84.2)
- moved D12 459.9 mm to (71.1, 14.0), turned to 90 degrees
- moved D41 435.7 mm to (38.9, 52.1), turned to 90 degrees
- moved D13 433.8 mm to (56.8, 14.0), turned to 90 degrees
- moved D11 423.4 mm to (94.9, 14.0), turned to 90 degrees
- moved D40 407.3 mm to (61.5, 52.1), turned to 90 degrees
- moved D4 397.8 mm to (228.2, 14.0), turned to 90 degrees
- moved D39 394.5 mm to (80.6, 52.1), turned to 90 degrees
- moved D10 383.9 mm to (113.9, 14.0), turned to 90 degrees
- moved D3 380.4 mm to (246.1, 14.0), turned to 90 degrees
- moved J5 375.6 mm to (280.9, 67.6), turned to 90 degrees
- moved DRST1 371.8 mm to (251.8, 69.7), turned to 270 degrees
- moved D26 370.8 mm to (66.3, 23.5), turned to 270 degrees
- moved D38 369.8 mm to (99.6, 52.1), turned to 90 degrees
- moved D43 364.4 mm to (242.5, 60.4), turned to 270 degrees
- moved D8 363.7 mm to (152.0, 14.0), turned to 90 degrees
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- renumbered D61 to D62
Connections:
- D15 pad 1: Net-(D15-Pad1) -> Row2
- D62 pad 1: Net-(D61-Pad1) -> Row4
- D62 pad 2: Net-(D61-Pad2) -> Net-(D62-Pad2)
- J5 pad 1: GND -> NRST
- J5 pad 2: NRST -> SWCLK
- J5 pad 5: SWCLK -> 3.3V
- J5 pad 6: 3.3V -> GND
- SW58 pad 1: Col9 -> Col10
- SW59 pad 1: Col10 -> Col11
- SW60 pad 1: Col11 -> Col12
- SW61 pad 1: Col13 -> Col12
- SW61 pad 2: Net-(D61-Pad2) -> Net-(D53-Pad2)
- SW62 pad 1: Col12 -> Col13
- SW62 pad 2: Net-(D53-Pad2) -> Net-(D62-Pad2)
- U1 pad 20: Net-(U1-Pad20) -> J3_1
- U1 pad 21: Net-(U1-Pad21) -> J3_2
- U1 pad 22: Net-(U1-Pad22) -> J3_3
- U1 pad 25: Net-(U1-Pad25) -> J3_4
- U1 pad 26: Net-(U1-Pad26) -> J3_5
- U1 pad 27: Net-(U1-Pad27) -> J3_6
- U1 pad 28: Net-(U1-Pad28) -> J2_1
- U1 pad 29: Net-(U1-Pad29) -> J2_2
- U1 pad 30: Net-(U1-Pad30) -> J2_3
- U1 pad 31: Net-(U1-Pad31) -> J2_4
- U1 pad 38: Net-(U1-Pad38) -> J2_5
- U1 pad 39: Net-(U1-Pad39) -> J2_6
Routing:
- net Net-(U1-Pad42): track 0.00 -> 324.5 mm
- net Row5: track 0.00 -> 303.6 mm
- net Net-(U1-Pad43): track 0.00 -> 282.0 mm
- net Row3: track 0.00 -> 268.0 mm
- net Row2: track 0.00 -> 263.6 mm
- net Col7: track 0.00 -> 255.2 mm
- net Row1: track 0.00 -> 249.1 mm
- net Net-(U1-Pad45): track 0.00 -> 241.2 mm
- net 3.3V: track 0.00 -> 229.6 mm, vias 0 -> 6
- net Col8: track 0.00 -> 217.5 mm
- net Row4: track 0.00 -> 214.8 mm
- net Net-(U1-Pad46): track 0.00 -> 209.7 mm
- net Net-(U1-Pad2): track 0.00 -> 185.9 mm
- net Col1: track 0.00 -> 185.5 mm
- net Col6: track 0.00 -> 183.9 mm
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- added copper zone on B.Cu, net /SHIELD
Other:
- outline, holes or cut-outs redrawn
- net class Default: trace_width 0.25 -> 0.254
- net class MCU  added: clearance 0.246, trace_width 0.254, via_dia 0.8, via_drill 0.4

Commit message: [Update] Finished routing
Parts:
- moved L1 57.0 mm to (178.1, 85.2)
- moved D5 1.96 mm to (202.8, 12.8)
- moved D10 1.19 mm to (113.9, 12.8)
- moved D11 1.19 mm to (94.9, 12.8)
- moved D12 1.19 mm to (71.1, 12.8)
- moved D13 1.19 mm to (56.8, 12.8)
- moved D14 1.19 mm to (35.3, 12.8)
- moved D2 1.19 mm to (249.7, 12.8)
- moved D3 1.19 mm to (246.1, 12.8)
- moved D4 1.19 mm to (228.2, 12.8)
- moved D6 1.19 mm to (190.1, 12.8)
- moved D7 1.19 mm to (171.1, 12.8)
- moved D8 1.19 mm to (152.0, 12.8)
- moved D9 1.19 mm to (133.0, 12.8)
Connections:
- J5 pad 2: SWCLK -> BOOT0
- J5 pad 3: BOOT0 -> SWCLK
- J5 pad 5: 3.3V -> GND
- J5 pad 6: GND -> 3.3V
Routing:
- net Col11: track 121.8 -> 415.8 mm
- net Col10: track 162.9 -> 438.4 mm
- net Col12: track 80.7 -> 347.4 mm
- net Col7: track 255.2 -> 508.5 mm
- net Col13: track 37.3 -> 239.1 mm
- net Col3: track 81.5 -> 190.7 mm
- net Col2: track 36.3 -> 125.3 mm
- net Col8: track 217.5 -> 265.5 mm
- net Col9: track 181.7 -> 226.3 mm
- net Col6: track 183.9 -> 227.9 mm
- net Col5: track 146.2 -> 188.3 mm
- net Col4: track 114.6 -> 153.0 mm
- net Row4: track 214.8 -> 251.0 mm
- net Col14: track 19.9 -> 40.8 mm
- net Net-(D53-Pad2): track 6.35 -> 23.3 mm
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Other:
- outline, holes or cut-outs redrawn
- net class Col4 added: clearance 0.254, trace_width 0.254, via_dia 0.8, via_drill 0.4
- net class Col5 added: clearance 0.254, trace_width 0.254, via_dia 0.8, via_drill 0.4
- net class Col6 added: clearance 0.254, trace_width 0.254, via_dia 0.8, via_drill 0.4
- net class Col7 added: clearance 0.254, trace_width 0.254, via_dia 0.8, via_drill 0.4
- net class Col8 added: clearance 0.254, trace_width 0.254, via_dia 0.8, via_drill 0.4
- net class Col9 added: clearance 0.254, trace_width 0.254, via_dia 0.8, via_drill 0.4

Commit message: [Update] Finished routing
Parts:
- moved L2 1.19 mm to (117.5, 85.4)
- moved L3 1.19 mm to (177.0, 85.4)
- moved CSO1 0.20 mm to (248.6, 71.2)
Connections:
- U1 pad 10: Net-(U1-Pad10) -> Col7
- U1 pad 11: Net-(U1-Pad11) -> Col6
- U1 pad 12: Net-(U1-Pad12) -> Col5
- U1 pad 13: Net-(U1-Pad13) -> Col4
- U1 pad 14: Net-(U1-Pad14) -> Col3
- U1 pad 15: Net-(U1-Pad15) -> Col2
- U1 pad 16: Net-(U1-Pad16) -> Row3
- U1 pad 17: Net-(U1-Pad17) -> Row4
- U1 pad 18: Net-(U1-Pad18) -> Col1
- U1 pad 19: Net-(U1-Pad19) -> Row5
- U1 pad 2: Net-(U1-Pad2) -> Col11
- U1 pad 3: Net-(U1-Pad3) -> Col10
- U1 pad 41: Net-(U1-Pad41) -> Row2
- U1 pad 42: Net-(U1-Pad42) -> Row1
- U1 pad 43: Net-(U1-Pad43) -> Col14
- U1 pad 45: Net-(U1-Pad45) -> Col13
- U1 pad 46: Net-(U1-Pad46) -> Col12
- U1 pad 5: Net-(U1-Pad5) -> Col9
- U1 pad 6: Net-(U1-Pad6) -> Col8
Routing:
- net Row1: track 250.1 -> 577.1 mm
- net Net-(U1-Pad42): track 324.5 -> 0.00 mm
- net Col14: track 40.8 -> 324.8 mm
- net Net-(U1-Pad43): track 282.0 -> 0.00 mm
- net Col13: track 239.1 -> 482.4 mm
- net Net-(U1-Pad45): track 241.2 -> 0.00 mm
- net Col12: track 347.4 -> 568.4 mm
- net Net-(U1-Pad46): track 209.7 -> 0.00 mm
- net Col11: track 415.8 -> 606.0 mm
- net Net-(U1-Pad2): track 185.9 -> 0.00 mm
- net Col10: track 438.4 -> 609.0 mm
- net Net-(U1-Pad3): track 166.8 -> 0.00 mm
- net Col9: track 226.3 -> 376.1 mm
- net Net-(U1-Pad5): track 148.4 -> 0.00 mm
- net Col8: track 265.5 -> 395.6 mm
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Other:
- net class Col4 removed
- net class Col5 removed
- net class Col6 removed
- net class Col7 removed
- net class Col8 removed
- net class Col9 removed
- net class Default: clearance 0.2 -> 0.127
- net class MCU  removed
- rule trace_clearance: 0.2 -> 0.127
- rule trace_min: 0.2 -> 0.254
- board text added: "3V3"
- board text added: "ArcticFoxPCB V. pre-Alpha Designed by Gondolindrim :dogwind:"
- board text added: "BOOT0"
- board text added: "GND"
- board text added: "NRST"
- board text added: "P20"
- board text added: "P21"
- board text added: "P22"
- board text added: "P25"
- board text added: "P26"
- board text added: "P27"
- board text added: "P28"
- board text added: "P29"
- board text added: "P30"
- board text added: "P31"
- board text added: "P38"
- board text added: "P39"
- board text added: "SWCLK"
- board text added: "SWDIO"
