File: kicadFiles/arcticPCB.kicad_pcb (KiCad board)
At the start: 2 copper layers, 283 x 94.2 mm, 174 parts, among them J1 TYPE-C-31-M12_13, J2 Conn_01x06_Male, J3 Conn_01x06_Male, J5 Conn_01x06_Male, SW1 MXSwitch, SW10 MXSwitch, SW11 MXSwitch, SW12 MXSwitch, SW13 MXSwitch, SW14 MXSwitch, SW15 MXSwitch, SW16 MXSwitch, SW17 MXSwitch, SW18 MXSwitch, SW19 MXSwitch, SW2 MXSwitch, SW20 MXSwitch, SW21 MXSwitch, SW22 MXSwitch, SW23 MXSwitch, SW24 MXSwitch, SW25 MXSwitch, SW26 MXSwitch, SW27 MXSwitch, SW28 MXSwitch, SW29 MXSwitch, SW3 MXSwitch, SW30 MXSwitch, SW31 MXSwitch, SW32 MXSwitch, SW33 MXSwitch, SW34 MXSwitch, SW35 MXSwitch, SW36 MXSwitch, SW37 MXSwitch, SW38 MXSwitch, SW39 MXSwitch, SW4 MXSwitch, SW40 MXSwitch, SW41 MXSwitch, SW42 MXSwitch, SW43 MXSwitch, SW44 MXSwitch, SW45 MXSwitch, SW46 MXSwitch, SW47 MXSwitch, SW48 MXSwitch, SW49 MXSwitch, SW5 MXSwitch, SW50 MXSwitch, SW51 MXSwitch, SW52 MXSwitch, SW53 MXSwitch, SW54 MXSwitch, SW55 MXSwitch, SW56 MXSwitch, SW57 MXSwitch, SW58 MXSwitch, SW59 MXSwitch, SW6 MXSwitch, SW60 MXSwitch, SW61 MXSwitch, SW62 MXSwitch, SW63 MXSwitch, SW64 MXSwitch, SW65 MXSwitch, SW7 MXSwitch, SW8 MXSwitch, SW9 MXSwitch, U1 STM32F072-LQFP48, U2 USBLC6-2SC6, U3 MCP1700-3302E_SOT23

Commit message: Add extra pins, organize schematic, add renders
- There were two pins in the PCB that were left unused and un-exposed to use. Now those two pins are broken out so they can be used. To execute this, some cols and rows had to have their pins reallocated.

- Schematic is better organized;

- Added KLE and PCB renders at the REAME file.
Parts:
- added J4: Conn_01x02, Connector_PinHeader_2.54mm:PinHeader_1x02_P2.54mm_Vertical, F.Cu at (282.2, 18.1)
- moved J2 3.81 mm to (282.2, 29.5)
- moved J3 3.81 mm to (282.2, 44.8)
- moved D1 0.76 mm to (280.6, 13.2)
Connections:
- U1 pad 2: Col11 -> Col12
- U1 pad 3: Col10 -> Col11
- U1 pad 4: Net-(U1-Pad4) -> Col10
- U1 pad 40: Net-(U1-Pad40) -> J4_2
- U1 pad 41: Row2 -> J4_1
- U1 pad 42: Row1 -> Row2
- U1 pad 43: Col14 -> Row1
- U1 pad 45: Col13 -> Col14
- U1 pad 46: Col12 -> Col13
Routing:
- net J4_1: track 0.00 -> 41.7 mm
- net J4_2: track 0.00 -> 37.3 mm
- net Col1: track 238.7 -> 221.5 mm
- net J2_4: track 37.5 -> 26.3 mm
- net J2_5: track 38.5 -> 31.6 mm
- net J2_6: track 39.9 -> 33.5 mm
- net J2_3: track 29.4 -> 24.6 mm
- net J3_2: track 34.0 -> 37.8 mm
- net J3_1: track 39.1 -> 42.5 mm
- net 3.3V: track 227.1 -> 223.9 mm
- net J3_4: track 22.6 -> 25.8 mm
- net J2_2: track 26.4 -> 23.4 mm
- net J3_3: track 31.8 -> 34.6 mm
- net Row3: track 284.8 -> 287.0 mm
- net D-: track 57.6 -> 59.6 mm
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Other:
- board text added: "P40"
- board text added: "P41"

Commit message: Optimize routing, move SWD pins
Parts:
- SW1, SW10, SW11, SW12, SW13, SW16, SW17, SW18, SW19, SW2, SW20, SW21, SW22, SW23, SW24, SW25, SW26, SW27, SW3, SW30, SW31, SW32, SW33, SW34, SW35, SW36, SW37, SW38, SW39, SW4, SW40, SW43, SW44, SW45, SW46, SW47, SW48, SW49, SW5, SW50, SW51, SW52, SW55, SW59, SW6, SW61, SW64, SW65, SW7, SW8, SW9: footprint acheron_MX:MX100 -> acheron_MX_SolderMask:MX100
- SW14: footprint acheron_MX:MX200 -> acheron_MX_SolderMask:MX200
- SW15, SW28, SW54, SW56, SW58, SW60: footprint acheron_MX:MX150 -> acheron_MX_SolderMask:MX150
- SW29, SW62: footprint acheron_MX:MX175 -> acheron_MX_SolderMask:MX175
- SW41, SW42: footprint acheron_MX:MX225 -> acheron_MX_SolderMask:MX225
- SW53: footprint acheron_MX:MX275 -> acheron_MX_SolderMask:MX275
- SW57: footprint acheron_MX:MX700R -> acheron_MX_SolderMask:MX700R
- SW63: footprint acheron_MX:MX125 -> acheron_MX_SolderMask:MX125
- moved L3 64.5 mm to (136.8, 35.0)
- moved J5 49.2 mm to (236.6, 89.0)
- moved L1 4.49 mm to (173.6, 85.4)
Connections:
- J5 pad 5: GND -> 3.3V
- J5 pad 6: 3.3V -> GND
Routing:
- net Col11: track 603.9 -> 392.3 mm
- net Col12: track 563.5 -> 373.2 mm
- net Col13: track 481.7 -> 324.3 mm
- net Col10: track 606.6 -> 450.6 mm
- net Row5: track 313.4 -> 390.6 mm
- net 3.3V: track 223.9 -> 183.1 mm, vias 6 -> 5
- net Col7: track 621.4 -> 585.9 mm
- net SWDIO: track 66.6 -> 92.9 mm
- net SWCLK: track 64.1 -> 87.9 mm
- net BOOT0: track 103.0 -> 126.8 mm, vias 2 -> 1
- net Col1: track 221.5 -> 197.8 mm
- net Col8: track 395.6 -> 386.9 mm
- net Col9: track 378.1 -> 370.4 mm
- net 5V: track 97.5 -> 92.9 mm
- net NRST: track 99.6 -> 102.7 mm
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Other:
- outline, holes or cut-outs redrawn

Commit message: Reorganize graphics, optimize routing
- The ./graphics folder was reorganized

- Some traces, specially the ones leading to SWD pins, were re-done for
efficiency and optimization
Parts:
- added L4: ArcticLabel, arcticGraphics:arcticLabel, F.Cu at (173.5, 85.4)
- added L5: Acheron Logo, arcticGraphics:arcticLabelMask, F.Cu at (173.5, 85.4)
- moved L3 2.14 mm to (138.9, 35.0)
Routing:
- net 3.3V: track 183.1 -> 144.6 mm
- net Col2: track 143.2 -> 134.6 mm
- net Row5: track 390.6 -> 398.7 mm
- net NRST: track 102.7 -> 98.3 mm
Other:
- board text removed: "ArcticFoxPCB V. pre-Alpha Designed by Gondolindrim :dogwind:"

Commit message: Update Library, improve footprints and label
- The label  was previously written "release Alpha" which is not the case (this is still version pre-Alpha);

- New MX_SolderMask witch footprints from the AcheronLibrary

- The extra pins were allocated into three symbols (J2, J3 and J4). These were grouped under the same J2, having 14 pins and an improved footprint;

- Optimized routing near the MCU area;

- Added more clearance to the D+/D- differential pair to make sure it is free from interference;
Parts:
- removed J3: Conn_01x06_Male, acheron_Connectors:HEADER_6PIN
- removed J4: Conn_01x02, Connector_PinHeader_2.54mm:PinHeader_1x02_P2.54mm_Vertical
- J2: value Conn_01x06_Male -> Conn_01x14; footprint acheron_Connectors:HEADER_6PIN -> Connector_PinHeader_2.54mm:PinHeader_1x14_P2.54mm_Vertical
- moved J2 11.4 mm to (282.3, 18.1), turned to 0 degrees
Connections:
- J2 pad 1: J2_1 -> J4_1
- J2 pad 2: J2_2 -> J4_2
- J2 pad 3: J2_3 -> J2_6
- J2 pad 4: J2_4 -> J2_5
- J2 pad 5: J2_5 -> J2_4
- J2 pad 6: J2_6 -> J2_3
Routing:
- net Col1: track 197.8 -> 209.4 mm
- net J2_4: track 26.3 -> 25.6 mm
Other:
- net class DiffPair added: clearance 0.508, trace_width 0.254, via_dia 0.8, via_drill 0.4

Commit message: Add new pin header footprints
- The AcheronLibrary pin header footprints were updated, and a SWD JTAG
footprint was added (see AcheronLibrary commit 280b825).

- Following this, the pin header footprints on Arctic were redone and
the JTAG footprint was added.
Parts:
- removed J5: Conn_01x06_Male, acheron_Connectors:HEADER_6PIN_HORIZONTAL
- added J3: Conn_ARM_JTAG_SWD_10, acheron_Connectors:Conn_ARM_JTAG_SWD_10, F.Cu at (304.3, 148.5)
- J2: footprint Connector_PinHeader_2.54mm:PinHeader_1x14_P2.54mm_Vertical -> acheron_Connectors:PinHeader_1x14_P2.54mm_Vertical
- moved J2 105.3 mm to (351.3, 97.7)
- moved CB4 93.5 mm to (332.3, 97.0)
- moved CRST1 93.5 mm to (325.7, 132.7)
- moved CUSB1 93.5 mm to (337.7, 78.9)
- moved D15 93.5 mm to (334.2, 86.6)
- moved D16 93.5 mm to (323.5, 86.6)
- moved D19 93.5 mm to (268.7, 86.6)
- moved D2 93.5 mm to (318.7, 75.9)
- moved D30 93.5 mm to (321.1, 115.2)
- moved D42 93.5 mm to (334.2, 122.3)
- moved D55 93.5 mm to (324.7, 142.6)
- moved F1 93.5 mm to (341.0, 78.0)
- moved H2 93.5 mm to (329.4, 91.4)
- moved H7 93.5 mm to (330.0, 148.3)
- moved J1 93.5 mm to (336.5, 70.9)
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Connections:
- net J2_1 renamed Extra8
- net J2_2 renamed Extra7
- net J2_3 renamed Extra6
- net J2_4 renamed Extra5
- net J2_5 renamed Extra4
- net J2_6 renamed Extra3
- net J3_1 renamed Extra14
- net J3_2 renamed Extra13
- net J3_3 renamed Extra12
- net J3_4 renamed Extra11
- net J3_5 renamed Extra10
- net J3_6 renamed Extra9
- net J4_1 renamed Extra1
- net J4_2 renamed Extra2
Routing:
- net BOOT0: track 126.8 -> 40.2 mm, vias 1 -> 2
- net Col1: track 209.4 -> 182.3 mm
- net 3.3V: track 144.6 -> 156.0 mm
- net Row5: track 398.7 -> 387.8 mm
- net Net-(D56-Pad2): track 6.25 -> 16.4 mm
- net NRST: track 98.3 -> 88.4 mm
- net SWDIO: track 92.9 -> 98.2 mm
- net SWCLK: track 87.9 -> 92.9 mm
- net 5V: track 92.9 -> 97.1 mm
- net Net-(D1-Pad2): track 8.50 -> 4.55 mm
- net VBUS: track 32.8 -> 31.4 mm
Other:
- outline, holes or cut-outs redrawn
- board text removed: "3V3"
- board text removed: "BOOT0"
- board text removed: "GND"
- board text removed: "NRST"
- board text removed: "SWCLK"
- board text removed: "SWDIO"

Commit message: Improved diff. pair pad clearances
- The differential pair D-/D+ has a 20thou clearance, which was used by
KiCad for the pads on USBLC6 (U2) and the microprocessor (U1), making
the filled zones around those pads not so good. The net clearance of
20thou remains, although the pads now have a normal clearance of 6 thou.
Parts:
- moved CSO1 19.1 mm to (318.9, 153.4)
- moved D17 19.1 mm to (308.1, 105.6)
- moved D20 19.1 mm to (250.9, 105.6)
- moved D22 19.1 mm to (212.8, 105.6)
- moved D23 19.1 mm to (193.8, 105.6)
- moved D25 19.1 mm to (155.7, 105.6)
- moved D26 19.1 mm to (136.6, 105.6)
- moved D27 19.1 mm to (117.6, 105.6)
- moved D28 19.1 mm to (85.4, 104.5)
- moved D29 19.1 mm to (335.4, 135.3)
- moved D43 19.1 mm to (312.8, 142.6)
- moved D47 19.1 mm to (236.6, 142.6)
- moved D48 19.1 mm to (217.6, 142.6)
- moved D51 19.1 mm to (160.4, 142.6)
- moved D52 19.1 mm to (141.4, 142.6)
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Routing:
- net Col13: track 324.3 -> 328.4 mm
- net Extra4: track 30.7 -> 32.0 mm
- net Extra1: track 39.5 -> 38.5 mm
- net Extra5: track 25.6 -> 26.6 mm
- net Extra2: track 34.3 -> 35.0 mm
- net Extra3: track 31.4 -> 32.0 mm
Other:
- board text added: "(I) If you want to check or reroute a specific trace, it is recommended that you use the High Contrast mode. Turn it on at View > Contrast mode > Check "High Contrast Mode". The icon is also available at the left icon column."
- board text added: "(II) It is recommended that the user has some knowledge in Git usage, since it is the main VCS tool used for the Acheron Project."
- board text added: "(III) All footprints are available either through KiCad's native libraries or the Acheron Library (http://github.com/Gondolindrim/AcheronLibrary). To facilitate the portability of the Acheron projects, this library is generally added at the ${KIPRJMOD} folder as a Git submodule. Hence, right after cloning the PCB repository, run: $ git submodules init --update To update the submodules."
- board text added: "(IV) For detailed information, check the Acheron Docs page for the ArcticPCB: http://gondolindrim.github.io/AcheronDocs/arctic/intro.html"
- board text added: "(i) The grid unit (1U) value used was 3/4" = 19.05mm"
- board text added: "(ii) The PCB was designed to fit the standards of the PCBWay manufacturer, at their cheapest settings."
- board text added: "(iii) All parts were quoted on the LCSC supplier (https://lcsc.com)."
- board text added: "(iv) You can always contact Gondolindrim through:"
- board text added: "(v) Most manufacturers list minimum character height as 0.8mm, and warn that any words using values below that will be undiscernable or unreadable. I have found that values down to 0.6mm (25 thou) can be used, although at that level a really close look is needed. Indeed, the minimum character height at which characters are easily readable is 0.8mm"
- board text added: "- ArcticPCB's GitHub page: http://github.com/Gondolindrim/ArcticPCB"
- board text added: "- Discord: Gondolindrim#9738"
- board text added: "- E-mail: alvaro.augusto.volpato@gmail.com"
- board text added: "- Reddit: /u/gondolindrim"
- board text added: "Also be sure to check with your parts supplier if they have all the necessary parts in the Bill of Materials and change parts and footprints accordingly to availability"
- board text added: "Be aware that capabilities may vary among manufacturers, so be sure to check with your manufacturer if they support the minimum values used."
- board text added: "GENERAL OBSERVATIONS"
- board text added: "MINIMUM CLEARANCE: 6 thou"
- board text added: "MINIMUM CLEARANCE: 8 thou"
- board text added: "MINIMUM VALUES"
- board text added: "RECOMMENDED VALUES"
- board text added: "SILKSCREEN CHARACTER HEIGHT: 25 thou (see General Observation (v))"
- board text added: "SILKSCREEN CHARACTER HEIGHT: 32 thou"
- board text added: "SILKSCREEN CHARACTER TRACE WIDTH: 6 thou"
- board text added: "SILKSCREEN CHARACTER TRACE WIDTH: 8 thou"
- board text added: "TRACE WIDTH: 10 thou"
- board text added: "TRACE WIDTH: 6 thou (approx. 0.15 mm)"
- board text added: "TRACE-TO-EDGE AND VIA-TO-EDGE DISTANCE: 8 thou"
- board text added: "These are general hints to use this PCB file. They are aimed specially at thoise new to KiCad or ECAD in general and to whoever wishes to use this project."
- board text added: "These values were the default values used when possible."
- board text added: "USAGE GUIDE (PLEASE READ)"
- board text added: "VIA DIAMETER: 20 thou (approx. 0.5mm)"
- board text added: "VIA DIAMETER: 32 thou (approx. 0.8mm)"
- board text added: "VIA HOLE SIZE: 12 thou (approx. 0.3mm)"
- board text added: "VIA HOLE SIZE: 16 thou (approx. 0.4mm)"
- board text added: "VIA-TO-VIA AND VIA-TO-TRACE CLEARANCE: 6 thou"
- board text added: "VIA-TO-VIA AND VIA-TO-TRACE CLEARANCE: 8 thou"
